File: PCB/analog sound synth.kicad_sch (KiCad schematic)
At the start: 0 parts

Commit message: work session 1
worked on button sub schematic and created rough design for op amp
square wave oscillators without precise values
Other:
- added sheet buttons ig (buttons.kicad_sch)
- added sheet power (power.kicad_sch)
- added sheet sq wave generators (sq wave generators.kicad_sch)
Changed lines of the file:
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@@
 	(generator_version "10.0")
 	(paper "A4")
+	(sheet
+		(at 83.82 22.86)
+		(size 43.18 22.86)
+		(exclude_from_sim no)
+		(in_bom yes)
+		(on_board yes)
+		(dnp no)
+		(fields_autoplaced yes)
+		(stroke
+			(width 0.1524)
+			(type solid)
+		)
+		(fill
+			(color 0 0 0 0)
+		)
+		(property "Sheetname" "sq wave generators"
+			(at 83.82 22.1484 0)
+			(show_name no)
+			(do_not_autoplace no)
+			(effects
+				(font
+					(size 1.27 1.27)
+				)
+				(justify left bottom)
+			)
+		)
+		(property "Sheetfile" "sq wave generators.kicad_sch"
+			(at 83.82 46.3046 0)
+			(show_name no)
+			(do_not_autoplace no)
+			(effects
+				(font
+					(size 1.27 1.27)
+				)
+				(justify left top)
+			)
+		)
+		(instances
+			(project "analog sound synth"
+				(path "/425447dc-c662-4463-a318-9ca8a58ab54a"
+					(page "4")
+				)
+			)
+		)
+	)
+	(sheet
+		(at 30.48 22.86)
+		(size 27.94 21.59)
+		(exclude_from_sim no)
+		(in_bom yes)
+		(on_board yes)
+		(dnp no)
+		(fields_autoplaced yes)
+		(stroke
+			(width 0.1524)
+			(type solid)
+		)
+		(fill
+			(color 0 0 0 0)
+		)
+		(property "Sheetname" "power"
+			(at 30.48 22.1484 0)
+			(show_name no)
+			(do_not_autoplace no)
+			(effects
+				(font
+					(size 1.27 1.27)
+				)
+				(justify left bottom)
+			)
+		)
+		(property "Sheetfile" "power.kicad_sch"
+			(at 30.48 45.0346 0)
+			(show_name no)
+			(do_not_autoplace no)
+			(effects
+				(font
+					(size 1.27 1.27)
+				)
+				(justify left top)
+			)
+		)
+		(instances
+			(project "analog sound synth"
+				(path "/425447dc-c662-4463-a318-9ca8a58ab54a"
+					(page "2")
+				)
+			)
+		)
+	)
+	(sheet
+		(at 29.21 62.23)
+		(size 33.02 29.21)
+		(exclude_from_sim no)
+		(in_bom yes)
+		(on_board yes)
+		(dnp no)
+		(fields_autoplaced yes)
+		(stroke
+			(width 0.1524)
+			(type solid)
+		)
+		(fill
+			(color 0 0 0 0)
+		)
+		(property "Sheetname" "buttons ig"
+			(at 29.21 61.5184 0)
+			(show_name no)
+			(do_not_autoplace no)
+			(effects
+				(font
+					(size 1.27 1.27)
+				)
+				(justify left bottom)
+			)
+		)
+		(property "Sheetfile" "buttons.kicad_sch"
+			(at 29.21 92.0246 0)
+			(show_name no)
+			(do_not_autoplace no)
+			(effects
+				(font
+					(size 1.27 1.27)
+				)
+				(justify left top)
+			)
+		)
+		(instances
+			(project "analog sound synth"
+				(path "/425447dc-c662-4463-a318-9ca8a58ab54a"
+					(page "3")
+				)
+			)
+		)
+	)
 	(sheet_instances
 		(path "/"

Commit message: I hate this
so much
Other:
- added sheet audio amplifier (audio amplifier.kicad_sch)
- added sheet audio summing integrator (audio summing integrator.kicad_sch)
- note added: "I dont know how to use hierarchal sheets gng"
Changed lines of the file:
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@@
 	(generator_version "10.0")
 	(paper "A4")
-	(sheet
-		(at 83.82 22.86)
+	(text "I dont know how to use hierarchal sheets gng"
+		(exclude_from_sim no)
+		(at 88.392 18.288 0)
+		(effects
+			(font
+				(size 1.27 1.27)
+			)
+		)
+	)
+	(sheet
+		(at 77.47 26.67)
 		(size 43.18 22.86)
 		(exclude_from_sim no)
@@
 		)
 		(property "Sheetname" "sq wave generators"
-			(at 83.82 22.1484 0)
+			(at 77.47 25.9584 0)
 			(show_name no)
 			(do_not_autoplace no)
@@
 		)
 		(property "Sheetfile" "sq wave generators.kicad_sch"
-			(at 83.82 46.3046 0)
+			(at 77.47 50.1146 0)
 			(show_name no)
 			(do_not_autoplace no)
@@
 	)
 	(sheet
-		(at 30.48 22.86)
+		(at 132.08 29.21)
+		(size 30.48 24.13)
+		(exclude_from_sim no)
+		(in_bom yes)
+		(on_board yes)
+		(dnp no)
+		(fields_autoplaced yes)
+		(stroke
+			(width 0.1524)
+			(type solid)
+		)
+		(fill
+			(color 0 0 0 0)
+		)
+		(property "Sheetname" "audio amplifier"
+			(at 132.08 28.4984 0)
+			(show_name no)
+			(do_not_autoplace no)
+			(effects
+				(font
+					(size 1.27 1.27)
+				)
+				(justify left bottom)
+			)
+		)
+		(property "Sheetfile" "audio amplifier.kicad_sch"
+			(at 132.08 53.9246 0)
+			(show_name no)
+			(do_not_autoplace no)
+			(effects
+				(font
+					(size 1.27 1.27)
+				)
+				(justify left top)
+			)
+		)
+		(instances
+			(project "analog sound synth"
+				(path "/425447dc-c662-4463-a318-9ca8a58ab54a"
+					(page "6")
+				)
+			)
+		)
+	)
+	(sheet
+		(at 85.09 67.31)
+		(size 46.99 31.75)
+		(exclude_from_sim no)
+		(in_bom yes)
+		(on_board yes)
+		(dnp no)
+		(fields_autoplaced yes)
+		(stroke
+			(width 0.1524)
+			(type solid)
+		)
+		(fill
+			(color 0 0 0 0)
+		)
+		(property "Sheetname" "audio summing integrator"
+			(at 85.09 66.5984 0)
+			(show_name no)
+			(do_not_autoplace no)
+			(effects
+				(font
+					(size 1.27 1.27)
+				)
+				(justify left bottom)
+			)
+		)
+		(property "Sheetfile" "audio summing integrator.kicad_sch"
+			(at 85.09 99.6446 0)
+			(show_name no)
+			(do_not_autoplace no)
+			(effects
+				(font
+					(size 1.27 1.27)
+				)
+				(justify left top)
+			)
+		)
+		(instances
+			(project "analog sound synth"
+				(path "/425447dc-c662-4463-a318-9ca8a58ab54a"
+					(page "5")
+				)
+			)
+		)
+	)
+	(sheet
+		(at 38.1 26.67)
 		(size 27.94 21.59)
 		(exclude_from_sim no)
@@
 		)
 		(property "Sheetname" "power"
-			(at 30.48 22.1484 0)
+			(at 38.1 25.9584 0)
 			(show_name no)
 			(do_not_autoplace no)
@@
 		)
 		(property "Sheetfile" "power.kicad_sch"
-			(at 30.48 45.0346 0)
+			(at 38.1 48.8446 0)
 			(show_name no)
 			(do_not_autoplace no)
@@
 	)
 	(sheet
-		(at 29.21 62.23)
-		(size 33.02 29.21)
+		(at 38.1 68.58)
+		(size 36.83 29.21)
 		(exclude_from_sim no)
 		(in_bom yes)
@@
 		)
 		(property "Sheetname" "buttons ig"
-			(at 29.21 61.5184 0)
+			(at 38.1 67.8684 0)
 			(show_name no)
 			(do_not_autoplace no)
@@
 		)
 		(property "Sheetfile" "buttons.kicad_sch"
-			(at 29.21 92.0246 0)
-			(show_name no)
-			(do_not_autoplace no)
+			(at 38.1 98.3746 0)
+			(show_name no)
+			(do_not_autoplace no)
