File: PCB/buttons.kicad_sch (KiCad schematic)
At the start: 20 parts, among them SW10 F4, SW11 F#4, SW12 G4, SW13 Ab4, SW14 A4, SW15 Bb4, SW16 B4, SW17 C5, SW18 C#5, SW19 D5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

Commit message: I hate this
so much
Connections:
- net A3 RC is gone; now on net A3 sq wave: SW2.6
- net A4 RC is gone; now on net A4 sq wave: SW14.6
- net Ab4 RC is gone; now on net Ab4 sq wave: SW13.6
- net B3 RC is gone; now on net B3 sq wave: SW4.6
- net B4 RC is gone; now on net B4 sq wave: SW16.6
- net Bb3 RC is gone; now on net Bb3 sq wave: SW3.6
- net Bb4 RC is gone; now on net Bb4 sq wave: SW15.6
- net C#4 RC is gone; now on net C#4 sq wave: SW6.6
- net C#5 RC is gone; now on net C#5 sq wave: SW18.6
- net C4 RC is gone; now on net C4 sq wave: SW5.6
- net C5 RC is gone; now on net C5 sq wave: SW17.6
- net D4 RC is gone; now on net D4 sq wave: SW7.6
- net D5 RC is gone; now on net D5 sq wave: SW19.6
- net E4 RC is gone; now on net E4 sq wave: SW9.6
- net E5 RC is gone; now on net E5 sq wave: SW21.6
- net Eb4 RC is gone; now on net Eb4 sq wave: SW8.6
- net Eb5 RC is gone; now on net Eb5 sq wave: SW20.6
- net F#4 RC is gone; now on net F#4 sq wave: SW11.6
- net F4 RC is gone; now on net F4 sq wave: SW10.6
- net G4 RC is gone; now on net G4 sq wave: SW12.6
- net A3 OPA: no longer SW2.2
- net A3 sq wave: no longer SW2.3
- net A4 OPA: no longer SW14.2
- net A4 sq wave: no longer SW14.3
- net Ab4 OPA: no longer SW13.2
- net Ab4 sq wave: no longer SW13.3
- net B3 OPA: no longer SW4.2
- net B3 sq wave: no longer SW4.3
- net B4 OPA: no longer SW16.2
- net B4 sq wave: no longer SW16.3
- net Bb3 OPA: no longer SW3.2
- net Bb3 sq wave: no longer SW3.3
- net Bb4 OPA: no longer SW15.2
- net Bb4 sq wave: no longer SW15.3
- net C#4 OPA: no longer SW6.2
- net C#4 sq wave: no longer SW6.3
- net C#5 OPA: no longer SW18.2
- net C#5 sq wave: no longer SW18.3
- net C4 OPA: no longer SW5.2
- net C4 sq wave: no longer SW5.3
- net C5 OPA: no longer SW17.2
- net C5 sq wave: no longer SW17.3
- net D4 OPA: no longer SW7.2
- net D4 sq wave: no longer SW7.3
- net D5 OPA: no longer SW19.2
- net D5 sq wave: no longer SW19.3
- net E4 OPA: no longer SW9.2
- net E4 sq wave: no longer SW9.3
- net E5 OPA: no longer SW21.2
- net E5 sq wave: no longer SW21.3
- net Eb4 OPA: no longer SW8.2
- net Eb4 sq wave: no longer SW8.3
- net Eb5 OPA: no longer SW20.2
- net Eb5 sq wave: no longer SW20.3
- net F#4 OPA: no longer SW11.2
- net F#4 sq wave: no longer SW11.3
- net F4 OPA: no longer SW10.2
- net F4 sq wave: no longer SW10.3
- net G4 OPA: no longer SW12.2
- net G4 sq wave: no longer SW12.3
- no-connect marks 40 -> 80
