File: PCB/sq wave generators.kicad_sch (KiCad schematic)
At the start: 110 parts, among them U1 LM358DR, U10 LM358DR, U2 LM358DR, U3 LM358DR, U4 LM358DR, U5 LM358DR, U6 LM358DR, U7 LM358DR, U8 LM358DR, U9 LM358DR

Commit message: I hate this
so much
Parts:
- removed U1, U10, U2, U3, U4, U5, U6, U7, U8, U9: LM358DR, EasyEDA:SOIC-8_L5.0-W4.0-P1.27-LS6.0-BL, symbol EasyEDA:LM358DR
- added C21, C22, C23, C24, C25, C26, C27, C28, C29, C30: 0.1uF, Capacitor_SMD:C_0402_1005Metric, symbol Device:C_Small
- added R115, R119, R120: 82k, Resistor_SMD:R_0603_1608Metric, symbol Device:R_Small_US
- added R116: 15k, Resistor_SMD:R_0402_1005Metric, symbol Device:R_Small_US
- added R117: 20k, Resistor_SMD:R_0402_1005Metric, symbol Device:R_Small_US
- added R118: 1.2k, Resistor_SMD:R_0402_1005Metric, symbol Device:R_Small_US
- added R121: 390, Resistor_SMD:R_0603_1608Metric, symbol Device:R_Small_US
- added R122: 62k, Resistor_SMD:R_0603_1608Metric, symbol Device:R_Small_US
- added R123: 6.2k, Resistor_SMD:R_0603_1608Metric, symbol Device:R_Small_US
- added R124: 820, Resistor_SMD:R_0603_1608Metric, symbol Device:R_Small_US
- added R125: 300k, Resistor_SMD:R_0402_1005Metric, symbol Device:R_Small_US
- added R126: 390k, Resistor_SMD:R_0603_1608Metric, symbol Device:R_Small_US
- added R81: 200k, Resistor_SMD:R_0402_1005Metric, symbol Device:R_Small_US
- added R82: 7.5k, Resistor_SMD:R_0402_1005Metric, symbol Device:R_Small_US
- added R83: 4.7k, Resistor_SMD:R_0402_1005Metric, symbol Device:R_Small_US
- added R84: 220, Resistor_SMD:R_0402_1005Metric, symbol Device:R_Small_US
- added R85: 3.3k, Resistor_SMD:R_0402_1005Metric, symbol Device:R_Small_US
- added R86: 2.2k, Resistor_SMD:R_0402_1005Metric, symbol Device:R_Small_US
- added R87: 510, Resistor_SMD:R_0402_1005Metric, symbol Device:R_Small_US
- added R88: 750k, Resistor_SMD:R_0603_1608Metric, symbol Device:R_Small_US
- added U1, U10, U2, U3, U4, U5, U6, U7, U8, U9: LM358DR2G, EasyEDA:SOIC-8_L5.0-W4.0-P1.27-LS6.0-BL, symbol EasyEDA:LM358DR2G
- C1, C10, C11, C12, C13, C14, C15, C16, C17, C18, C19, C2, C20, C3, C4, C5, C6, C7, C8, C9: value C_Small -> 10nF; footprint (none) -> Capacitor_SMD:C_0603_1608Metric
- R1, R40: value R_Small_US -> 180k; footprint (none) -> Resistor_SMD:R_0603_1608Metric
- R10, R13, R14, R17, R18, R21, R22, R25, R26, R28, R29, R3, R30, R33, R34, R37, R38, R4, R41, R42, R43, R44, R48, R49, R5, R50, R51, R52, R55, R57, R58, R6, R61, R62, R65, R66, R69, R70, R73, R74, R77, R78, R9: value R_Small_US -> 47k; footprint (none) -> Resistor_SMD:R_0402_1005Metric
- R11, R15, R19, R2, R23, R27, R31, R35, R39, R45, R46, R53, R54, R59, R63, R67, R7, R71, R75, R79: value R_Small_US -> 4.7k; footprint (none) -> Resistor_SMD:R_0402_1005Metric
- R12: value R_Small_US -> 2.4k; footprint (none) -> Resistor_SMD:R_0402_1005Metric
- R16, R20: value R_Small_US -> 75k; footprint (none) -> Resistor_SMD:R_0402_1005Metric
- R24: value R_Small_US -> 56k; footprint (none) -> Resistor_SMD:R_0402_1005Metric
- R32: value R_Small_US -> 62k; footprint (none) -> Resistor_SMD:R_0603_1608Metric
- R36: value R_Small_US -> 220k; footprint (none) -> Resistor_SMD:R_0402_1005Metric
- R47: value R_Small_US -> 51k; footprint (none) -> Resistor_SMD:R_0402_1005Metric
- R56: value R_Small_US -> 160k; footprint (none) -> Resistor_SMD:R_0603_1608Metric
- R60: value R_Small_US -> 36k; footprint (none) -> Resistor_SMD:R_0603_1608Metric
- R64, R72: value R_Small_US -> 39k; footprint (none) -> Resistor_SMD:R_0402_1005Metric
- R68: value R_Small_US -> 43k; footprint (none) -> Resistor_SMD:R_0603_1608Metric
- R76, R80: value R_Small_US -> 33k; footprint (none) -> Resistor_SMD:R_0402_1005Metric
- R8: value R_Small_US -> 82k; footprint (none) -> Resistor_SMD:R_0603_1608Metric
Connections:
- net +BATT: now also R33.2, R43.2, C21.1, C22.1, C23.1, C24.1, C25.1, C26.1, C27.1, C28.1, C29.1, C30.1, U1.8 (+V), U10.8 (+V), U2.8 (+V), U3.8 (+V), U4.8 (+V), U5.8 (+V), U6.8 (+V), U7.8 (+V), U8.8 (+V), U9.8 (+V)
- net -BATT: now also R34.1, R44.1, C21.2, C22.2, C23.2, C24.2, C25.2, C26.2, C27.2, C28.2, C29.2, C30.2, U1.4 (GND), U10.4 (GND), U2.4 (GND), U3.4 (GND), U4.4 (GND), U5.4 (GND), U6.4 (GND), U7.4 (GND), U8.4 (GND), U9.4 (GND)
- net A3 OPA: now also U1.1 (OUT1); no longer R11.2, R19.2, R27.2, R35.2, R45.2, R46.2, R59.2, R67.2, R75.2
- net Bb3 OPA: now also U1.7 (OUT2); no longer R15.2, R23.2, R31.2, R39.2, R53.2, R54.2, R63.2, R71.2, R79.2
- net at R29.1, R30.2, R31.1: now also U4.5 (+IN2)
- net at C8.2: now also R118.1, U4.6 (-IN2); no longer R32.1
- net at R28.1: now also R117.2; no longer C7.2
- net at R41.1, R42.2, R45.1: now also U6.3 (+IN1)
- net at R37.1, R38.2, R39.1: now also U5.5 (+IN2)
- net at C17.2, R68.1: now also R125.1, U9.2 (-IN1)
- net at R69.1, R70.2, R71.1: now also U9.5 (+IN2)
- net at R55.1: now also R85.2; no longer C13.2
- net at R33.1: now also R34.2, R35.1, U5.3 (+IN1)
- net at R13.1, R14.2, R15.1: now also U2.5 (+IN2)
- net at C4.2: now also R83.1, U2.6 (-IN2); no longer R16.1
- net at R8.1: now also R82.2; no longer C2.2
- net at R65.1, R66.2, R67.1: now also U9.3 (+IN1)
- net at C18.2, R72.1: now also R126.1, U9.6 (-IN2)
- net at C20.2, R80.1: now also R88.1, U10.6 (-IN2)
- net at R57.1, R58.2, R59.1: now also U8.3 (+IN1)
- net at C6.2: now also R116.1, U3.6 (-IN2); no longer R24.1
- net at R77.1, R78.2, R79.1: now also U10.5 (+IN2)
- net at C15.2: now also R123.1, U8.2 (-IN1); no longer R60.1
- net at R5.1, R6.2, R7.1: now also U1.5 (+IN2)
- net at R61.1, R62.2, R63.1: now also U8.5 (+IN2)
- net at C16.2, R64.1: now also U8.6 (-IN2)
- net at C3.2, R12.1: now also U2.2 (-IN1)
- net at R10.2, R11.1, R9.1: now also U2.3 (+IN1)
- net at C11.2: now also R86.1, U6.2 (-IN1); no longer R47.1
- net at C12.2, R48.1: now also U7.2 (-IN1)
- net at R49.1, R50.2, R53.1: now also U6.5 (+IN2)
- net at C9.2, R36.1: now also R119.1, U5.2 (-IN1)
- net at C19.2: now also R87.1, U10.2 (-IN1); no longer R76.1
- net at R73.1, R74.2, R75.1: now also U10.3 (+IN1)
- net at C5.2: now also R84.1, U3.2 (-IN1); no longer R20.1
- net at R17.1, R18.2, R19.1: now also U3.3 (+IN1)
- net at R21.1, R22.2, R23.1: now also U3.5 (+IN2)
- net at C14.2, R56.1: now also R122.1, U7.6 (-IN2)
- net at R25.1, R26.2, R27.1: now also U4.3 (+IN1)
- net at C1.2, R1.1: now also R81.1, U1.2 (-IN1)
- net at R46.1: now also R43.1, R44.2, U7.3 (+IN1)
- net at R2.1, R3.1, R4.2: now also U1.3 (+IN1)
- net at R51.1, R52.2, R54.1: now also U7.5 (+IN2)
- net at C10.2, R40.1: now also R120.1, U5.6 (-IN2)
- removed net A3 RC: R1.2, R12.2, R20.2, R28.2, R36.2, R47.2, R48.2, R60.2, R68.2, R76.2
- removed net Bb3 RC: R16.2, R24.2, R32.2, R40.2, R55.2, R56.2, R64.2, R72.2, R8.2, R80.2
- new net: R116.2, R24.1
- new net: R123.2, R60.1
- new net: C2.2, R82.1, U1.6 (-IN2)
- new net: C13.2, R85.1, U6.6 (-IN2)
- new net: R47.1, R86.2
- new net: R118.2, R32.1
- new net: R16.1, R83.2
- new net: R115.1, R12.2
- new net: R20.1, R84.2
- new net: C7.2, R117.1, U4.2 (-IN1)
- new net: R121.1, R48.2
- new net: R124.1, R64.2
- new net: R76.1, R87.2
- new net A3 sq wave: R1.2, R81.2
- new net A4 OPA: R46.2, U7.1 (OUT1)
- new net A4 sq wave: R121.2
- new net Ab4 OPA: R53.2, U6.7 (OUT2)
- new net Ab4 sq wave: R55.2
- new net B3 OPA: R11.2, U2.1 (OUT1)
- new net B3 sq wave: R115.2
- new net B4 OPA: R59.2, U8.1 (OUT1)
- new net B4 sq wave: R60.2
- new net Bb3 sq wave: R8.2
- new net Bb4 OPA: R54.2, U7.7 (OUT2)
- new net Bb4 sq wave: R122.2, R56.2
- new net C#4 OPA: R19.2, U3.1 (OUT1)
- new net C#4 sq wave: R20.2
- new net C#5 OPA: R67.2, U9.1 (OUT1)
- new net C#5 sq wave: R125.2, R68.2
- new net C4 OPA: R15.2, U2.7 (OUT2)
- new net C4 sq wave: R16.2
- new net C5 OPA: R63.2, U8.7 (OUT2)
- new net C5 sq wave: R124.2
- new net D4 OPA: R23.2, U3.7 (OUT2)
- new net D4 sq wave: R24.2
- new net D5 OPA: R71.2, U9.7 (OUT2)
- new net D5 sq wave: R126.2, R72.2
- new net E4 OPA: R31.2, U4.7 (OUT2)
- new net E4 sq wave: R32.2
- new net E5 OPA: R79.2, U10.7 (OUT2)
- new net E5 sq wave: R80.2, R88.2
- new net Eb4 OPA: R27.2, U4.1 (OUT1)
- new net Eb4 sq wave: R28.2
- new net Eb5 OPA: R75.2, U10.1 (OUT1)
- new net Eb5 sq wave: R76.2
- new net F#4 OPA: R39.2, U5.7 (OUT2)
- new net F#4 sq wave: R120.2, R40.2
- new net F4 OPA: R35.2, U5.1 (OUT1)
- new net F4 sq wave: R119.2, R36.2
- new net G4 OPA: R45.2, U6.1 (OUT1)
- new net G4 sq wave: R47.2
Other:
- moved on the sheet: C1, C11, C12, C15, C17, C19, C3, C5, C7, C9, R1, R12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
